File: 02 - CDRF/01 - ELECTRONIQUE/PUMP PCB/PCB PUMP.brd (EAGLE design)
At the start: 25 x 25 mm, 13 parts, among them J3 PWRPAD2-5MM, J4 PWRPAD2-5MM

Commit message: update
Parts:
- moved R2 9.71 mm to (8.31, 5.17), flipped to the bottom
- moved T1 3.06 mm to (7.11, 4.83)
- moved R1 2.97 mm to (10.7, 4.32)
- moved D2 0.72 mm to (3.37, 17.2), turned to 60 degrees
- moved R3 0.57 mm to (13.7, 4.32)
Routing:
- net N$3: track 14.5 -> 2.93 mm, vias 2 -> 0
- net PUMP: track 6.34 -> 0.00 mm
- net N$2: track 7.98 -> 12.7 mm
- net N$4: track 14.4 -> 11.8 mm
- net +5V: track 33.5 -> 32.9 mm
- removed copper zone on layer 1, net GND
- removed copper zone on layer 16, net GND
