File: 02 - CDRF/01 - ELECTRONIQUE/PUMP PCB/PCB PUMP LED SENSOR.brd (EAGLE design)
At the start: 25 x 25 mm, 19 parts, among them J3 PWRPAD2-5MM, J4 PWRPAD2-5MM

Commit message: update pcb pump
Parts:
- removed PAD3, PAD4: WIREPAD1,6/0,8, wirepad:1,6/0,8
- added IC1: AD8217BRMZ, AD8217BRMZ:SOP65P490X110-8N
- added R8: (no value), rcl:R0805
- added X1: 22-23-2051, con-molex:22-23-2051
- J1: value (none) -> 22-27-2021-02; device OPENBOT:MOLEX-1X4 -> con-molex:6410-02
- moved J1 15.6 mm to (17.5, 8.38), turned to 90 degrees
- moved R7 12.7 mm to (14.1, 17.8), turned to 180 degrees
- moved U$3 8.30 mm to (15.0, 13.5), turned to 270 degrees
- moved U$2 5.71 mm to (11.7, 13.5), turned to 270 degrees
- moved R4 5.34 mm to (11.4, 4.95)
- moved R1 3.59 mm to (6.60, 5.08), flipped to the bottom
- moved D2 2.30 mm to (2.35, 15.7), turned to 73 degrees
- moved U$1 2.29 mm to (18.3, 13.5), turned to 270 degrees
- moved T1 1.61 mm to (5.12, 5.87), turned to 213 degrees
- moved R2 1.57 mm to (9.07, 5.04)
- moved R5 1.30 mm to (19.6, 17.8), turned to 180 degrees
- moved R3 1.14 mm to (13.0, 4.32)
- moved T2 1.05 mm to (17.5, 3.81)
- moved R6 0.92 mm to (8.64, 17.8)
- moved D1 0.16 mm to (22.5, 9.00), turned to 71 degrees
Connections:
- removed net N$2: D2.A, J3.P$1, T1.1
- new net MOTOR-: D2.A, IC1.8, J3.P$1, R8.2, T1.1
- new net OUT_SENSOR: IC1.5, X1.4
- net +5V: now also IC1.1, R8.1, X1.5; no longer PAD3.1
- net EV: now also X1.2; no longer J1.3
- net GND: now also IC1.4, X1.1; no longer J1.4
- net N$1: now also J1.2; no longer PAD4.1
- net PUMP: now also X1.3; no longer J1.2
Routing:
- net MOTOR-: track 0.00 -> 14.8 mm
- net N$2: track 12.4 -> 0.00 mm
- net GND: track 11.7 -> 0.00 mm, vias 0 -> 1
- net OUT_SENSOR: track 0.00 -> 8.59 mm
- net EV: track 22.3 -> 16.3 mm
- net +5V: track 37.0 -> 31.5 mm, vias 0 -> 2
- net N$5: track 4.80 -> 8.46 mm
- net N$1: track 6.22 -> 9.17 mm
- net N$3: track 7.78 -> 10.7 mm
- net N$4: track 10.1 -> 9.00 mm
- net PUMP: track 17.3 -> 16.7 mm
- added copper zone on layer 16, net +5V
