File: 02 - CDRF/01 - ELECTRONIQUE/PUMP PCB/PCB PUMP LED SENSOR.sch (EAGLE design)
At the start: 19 parts, among them J3 PWRPAD2-5MM, J4 PWRPAD2-5MM

Commit message: update pcb pump
Parts:
- removed PAD3, PAD4: WIREPAD1,6/0,8, wirepad:WIREPAD1,6/0,8
- added IC1: AD8217BRMZ, AD8217BRMZ:AD8217BRMZ
- added R8: (no value), rcl:R-EU_R0805
- added X1: 22-23-2051, con-molex:22-23-2051
- J1: value (none) -> 22-27-2021-02; device OPENBOT:CONN_04POLAR -> con-molex:22-27-2021-02
Connections:
- removed net N$2: D2.A, J3.PWRPAD, T1.D
- new net MOTOR-: D2.A, IC1.-IN, J3.PWRPAD, R8.2, T1.D
- new net OUT_SENSOR: IC1.OUT, X1-4.S
- net +5V: now also IC1.+IN, J1-1.S, R8.1, X1-5.S; no longer J1.1, PAD3.P
- net EV: now also X1-2.S; no longer J1.3
- net GND: now also IC1.GND, X1-1.S; no longer J1.4
- net N$1: now also J1-2.S; no longer PAD4.P
- net PUMP: now also X1-3.S; no longer J1.2
