File: 02 - CDRF/01 - ELECTRONIQUE/PCB MAT BALISE/PCB MAT BALISE/PCB_MAT_BALISE.brd (EAGLE design)
At the start: 72 x 50 mm, 15 parts, among them U1 A000053

Commit message: update
Parts:
- added C1: (no value), rcl:E5-10,5
- added C2: (no value), rcl:E2,5-7
- added CAPTEUR_AR_SORTIE, CAPTEUR_AV_SORTIE, ORIENTATION_SORTIE: (no value), CONNECTORS:MOLEX-1X3
- added I2C, I2C1, I2C2, SERIAL: (no value), CONNECTORS:MOLEX-1X4
- added PS1: R-78E5.0-1.0, KARIBOUS:CONV_R-78E5.0-1.0
- added R8, R9: (no value), fab:R1206FAB
- added RU1: RUEF300, OPENBOT:RUEF300
- added U$1: CONN_02_PUI, OPENBOT:NSK396-2C
- moved CAPTEUR_AV 42.1 mm to (55.9, 41.9), turned to 270 degrees
- moved SERVO 39.5 mm to (58.4, 2.54), turned to 90 degrees
- moved D2 37.0 mm to (67.3, 29.2), turned to 180 degrees
- moved CAPTEUR_AR 36.9 mm to (49.5, 41.9), turned to 270 degrees
- moved D1 34.4 mm to (59.7, 45.7)
- moved R1 34.4 mm to (59.7, 35.6)
- moved D3 34.3 mm to (67.3, 21.6), turned to 180 degrees
- moved R6 32.5 mm to (29.2, 41.9), turned to 180 degrees
- moved R5 31.7 mm to (17.8, 41.9), turned to 180 degrees
- moved R7 30.3 mm to (40.6, 41.9), turned to 180 degrees
- moved R2 30.1 mm to (59.7, 24.1)
- moved R3 26.1 mm to (59.7, 20.3)
- moved D4 20.1 mm to (67.3, 36.8), turned to 180 degrees
- moved R4 15.3 mm to (59.7, 27.9)
Connections:
- new net +24V: C2.+, RU1.P$1, U$1.P$2
- new net CAPT_AR_SORTIE: CAPTEUR_AR_SORTIE.3, U1.10
- new net CAPT_AV_SORTIE: CAPTEUR_AV_SORTIE.3, U1.9
- new net N$10: U1.26
- new net N$5: PS1.1, RU1.P$2
- new net ORIENTATION_SORTIE: ORIENTATION_SORTIE.3, U1.11
- new net RX: SERIAL.3, U1.4
- new net SCL: I2C.3, I2C1.3, I2C2.3, R8.2, U1.8
- new net SDA: I2C.4, I2C1.4, I2C2.4, R9.1, U1.7
- new net TX: SERIAL.4, U1.3
- net +5V: now also C1.+, I2C.2, I2C1.2, I2C2.2, PS1.3, R8.1, R9.2, SERIAL.2
- net CAPT_AR: now also U1.22
- net CAPT_AV: now also U1.21
- net DETECT_AR: now also U1.17
- net DETECT_AV: now also U1.16
- net EMITT_1: now also U1.18
- net GND: now also C1.-, C2.-, CAPTEUR_AR_SORTIE.1, CAPTEUR_AV_SORTIE.1, I2C.1, I2C1.1, I2C2.1, ORIENTATION_SORTIE.1, PS1.2, SERIAL.1, U$1.P$1
- net SIGNAL_1: now also U1.24
- net SIGNAL_2: now also U1.25
- net SIGNAL_ORIENTATION: now also U1.15
- net SIGNAL_SERVO: now also U1.14
- net VITESSE_SERVO: now also U1.23

Commit message: routage
Parts:
- removed D1, D2, D3, D4: (no value), OPENBOT:LED_5MM
- removed I2C, I2C1: (no value), CONNECTORS:MOLEX-1X4
- added R10: (no value), fab:R1206FAB
- added U$2, U$3: CONN_05, CONNECTORS:MOLEX-1X5
- added U$4, U$5, U$6, U$7, U$8: LED, fab:LED1206
- C1: value (none) -> 470uF
- C2: value (none) -> 10uF
- moved R1 42.8 mm to (17.8, 26.7)
- moved ORIENTATION_SORTIE 11.4 mm to (40.6, 2.54)
- moved R4 7.73 mm to (61.0, 35.6)
- moved CAPTEUR_AR_SORTIE 7.62 mm to (53.3, 2.54)
- moved CAPTEUR_AV_SORTIE 7.62 mm to (47.0, 2.54)
- moved RU1 4.34 mm to (10.7, 22.5), turned to 90 degrees
- moved R2 4.02 mm to (61.0, 27.9)
- moved R3 4.02 mm to (61.0, 24.1)
- moved CAPTEUR_AR 3.81 mm to (45.7, 41.9)
- moved CAPTEUR_AV 3.81 mm to (52.1, 41.9)
- moved C1 2.84 mm to (68.6, 15.2)
- moved R5 2.54 mm to (15.2, 41.9)
- moved R6 2.54 mm to (26.7, 41.9)
- moved R7 2.54 mm to (38.1, 41.9)
- moved PS1 1.42 mm to (6.99, 34.3), turned to 0 degrees
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Connections:
- new net N$6: R10.1, U$4.1
- new net XSHUT_AR: U$2.5, U1.9
- new net XSHUT_AV: U$3.5, U1.10
- net +24V: now also R10.2; no longer C2.+
- net +5V: now also CAPTEUR_AR_SORTIE.2, CAPTEUR_AV_SORTIE.2, ORIENTATION_SORTIE.2, U$2.2, U$3.2; no longer I2C.2, I2C1.2
- net CAPT_AR_SORTIE: now also U1.13; no longer U1.10
- net CAPT_AV_SORTIE: now also U1.12; no longer U1.9
- net GND: now also U$2.1, U$3.1, U$4.2, U$5.2, U$6.2, U$7.2, U$8.2; no longer D1.K, D2.K, D3.K, D4.K, I2C.1, I2C1.1
- net N$1: now also U$5.1; no longer D1.A
- net N$2: now also U$6.1; no longer D2.A
- net N$3: now also U$7.1; no longer D3.A
- net N$4: now also U$8.1; no longer D4.A
- net N$5: now also C2.+
- net SCL: now also U$2.3, U$3.3; no longer I2C.3, I2C1.3
- net SDA: now also U$2.4, U$3.4; no longer I2C.4, I2C1.4
- net SIGNAL_ORIENTATION: now also U1.14; no longer U1.15
- net SIGNAL_SERVO: now also U1.15; no longer U1.14
Routing:
- net +5V: track 0.00 -> 226.0 mm
- net SIGNAL_2: track 0.00 -> 29.3 mm
- net SCL: track 0.00 -> 26.1 mm
- net SDA: track 0.00 -> 21.7 mm
- net SIGNAL_1: track 0.00 -> 20.1 mm
- net RX: track 0.00 -> 14.2 mm
- net DETECT_AV: track 0.00 -> 14.1 mm
- net SIGNAL_ORIENTATION: track 0.00 -> 14.1 mm
- net XSHUT_AR: track 0.00 -> 12.9 mm
- net +24V: track 0.00 -> 12.7 mm
- net N$5: track 0.00 -> 12.6 mm
- net CAPT_AR_SORTIE: track 0.00 -> 11.0 mm
- net TX: track 0.00 -> 11.0 mm
- net VITESSE_SERVO: track 0.00 -> 10.5 mm
- net SIGNAL_SERVO: track 0.00 -> 10.1 mm
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- added copper zone on layer 1, net GND
- added copper zone on layer 16, net GND
