File: 02 - CDRF/01 - ELECTRONIQUE/PCB MAT BALISE/PCB MAT BALISE/PCB_MAT_BALISE.sch (EAGLE design)
At the start: 15 parts, among them U1 A000053

Commit message: update
Parts:
- added C1: (no value), rcl:CPOL-EUE5-10.5
- added C2: (no value), rcl:CPOL-EUE2.5-7
- added CAPTEUR_AR_SORTIE, CAPTEUR_AV_SORTIE, ORIENTATION_SORTIE: (no value), CONNECTORS:CONN_03POLAR
- added I2C, I2C1, I2C2, SERIAL: (no value), CONNECTORS:CONN_04POLAR
- added PS1: R-78E5.0-1.0, KARIBOUS:R-78E5.0-1.0
- added R8, R9: (no value), fab:RES-US1206FAB
- added RU1: RUEF300, OPENBOT:RUEF300
- added U$1: CONN_02_PUI, OPENBOT:CONN_02_PUI
Connections:
- new net +24V: C2.+, RU1.P$1, U$1.V+/VCC
- new net CAPT_AR_SORTIE: CAPTEUR_AR_SORTIE.3, U1.5(PWM)
- new net CAPT_AV_SORTIE: CAPTEUR_AV_SORTIE.3, U1.4/A6
- new net N$10: U1.A5
- new net N$5: PS1.+VIN, RU1.P$2
- new net ORIENTATION_SORTIE: ORIENTATION_SORTIE.3, U1.6(PWM)/A7
- new net RX: SERIAL.3, U1.0/RX
- new net SCL: I2C.3, I2C1.3, I2C2.3, R8.2, U1.3(PWM)/SCL
- new net SDA: I2C.4, I2C1.4, I2C2.4, R9.1, U1.2/SDA
- new net TX: SERIAL.4, U1.1/TX
- net +5V: now also C1.+, I2C.2, I2C1.2, I2C2.2, PS1.+VOUT, R8.1, R9.2, SERIAL.2, U1.+5V
- net CAPT_AR: now also U1.A1
- net CAPT_AV: now also U1.A0
- net DETECT_AR: now also U1.12/A11
- net DETECT_AV: now also U1.11(PWM)
- net EMITT_1: now also U1.13(PWM)
- net GND: now also C1.-, C2.-, CAPTEUR_AR_SORTIE.1, CAPTEUR_AV_SORTIE.1, I2C.1, I2C1.1, I2C2.1, ORIENTATION_SORTIE.1, PS1.GND, SERIAL.1, U$1.GND/COM
- net SIGNAL_1: now also U1.A3
- net SIGNAL_2: now also U1.A4
- net SIGNAL_ORIENTATION: now also U1.10(PWM)/A10
- net SIGNAL_SERVO: now also U1.9(PWM)/A9
- net VITESSE_SERVO: now also U1.A2

Commit message: routage
Parts:
- removed D1, D2, D3, D4: (no value), OPENBOT:LED5MM
- removed I2C, I2C1: (no value), CONNECTORS:CONN_04POLAR
- added R10: (no value), fab:RES-US1206FAB
- added U$2, U$3: CONN_05, CONNECTORS:CONN_05
- added U$4, U$5, U$6, U$7, U$8: LED, fab:LED
- C1: value (none) -> 470uF
- C2: value (none) -> 10uF
Connections:
- new net N$6: R10.1, U$4.A
- new net XSHUT_AR: U$2.5, U1.4/A6
- new net XSHUT_AV: U$3.5, U1.5(PWM)
- net +24V: now also R10.2; no longer C2.+
- net +5V: now also CAPTEUR_AR_SORTIE.2, CAPTEUR_AV_SORTIE.2, ORIENTATION_SORTIE.2, U$2.2, U$3.2; no longer I2C.2, I2C1.2
- net CAPT_AR_SORTIE: now also U1.8/A8; no longer U1.5(PWM)
- net CAPT_AV_SORTIE: now also U1.7; no longer U1.4/A6
- net GND: now also U$2.1, U$3.1, U$4.C, U$5.C, U$6.C, U$7.C, U$8.C; no longer D1.C, D2.C, D3.C, D4.C, I2C.1, I2C1.1
- net N$1: now also U$5.A; no longer D1.A
- net N$2: now also U$6.A; no longer D2.A
- net N$3: now also U$7.A; no longer D3.A
- net N$4: now also U$8.A; no longer D4.A
- net N$5: now also C2.+
- net SCL: now also U$2.3, U$3.3; no longer I2C.3, I2C1.3
- net SDA: now also U$2.4, U$3.4; no longer I2C.4, I2C1.4
- net SIGNAL_ORIENTATION: now also U1.9(PWM)/A9; no longer U1.10(PWM)/A10
- net SIGNAL_SERVO: now also U1.10(PWM)/A10; no longer U1.9(PWM)/A9
Other:
- moved on the sheet: C2, RU1
