File: 02 - MAKERFIGHT/02 - ELECTRONIQUE/CARTE_PUISSANCE/CARTE_PUISSANCE.sch (EAGLE design)
At the start: 15 parts

Commit message: update
Parts:
- added D5: (no value), OPENBOT:LED5MM
- added R5: (no value), rcl:R-EU_0204/7
- added U$8: CONN_02_PUIXT60, OPENBOT:CONN_02_PUIXT60
- added U$9: AUTOMOTIVE_FUSE, OPENBOT:AUTOMOTIVE_FUSE
Connections:
- new net N$3: R5.2, U$8.V+/VCC, U$9.P$2
- new net N$9: D5.A, R5.1
- net +12V: now also U$9.P$1
- net GND: now also D5.C, U$8.GND/COM
Changed lines of the file:
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@@
 <setting verticaltext="up"/>
 </settings>
-<grid distance="0.05" unitdist="inch" unit="inch" style="lines" multiple="1" display="no" altdistance="0.01" altunitdist="inch" altunit="inch"/>
+<grid distance="0.1" unitdist="inch" unit="inch" style="lines" multiple="1" display="no" altdistance="0.01" altunitdist="inch" altunit="inch"/>
 <layers>
 <layer number="1" name="Top" color="4" fill="1" visible="no" active="no"/>
@@
 </classes>
 <parts>
-<part name="U$6" library="OPENBOT" library_urn="urn:adsk.eagle:library:760642" deviceset="CONN_02_PUI" device="XT60"/>
+<part name="U$6" library="OPENBOT" library_urn="urn:adsk.eagle:library:760642" deviceset="CONN_02_PUI" device="XT60" package3d_urn="urn:adsk.eagle:package:16508586/1"/>
 <part name="D1" library="OPENBOT" library_urn="urn:adsk.eagle:library:760642" deviceset="LED" device="5MM" package3d_urn="urn:adsk.eagle:package:760648/2"/>
 <part name="R1" library="rcl" library_urn="urn:adsk.eagle:library:334" deviceset="R-EU_" device="0204/7" package3d_urn="urn:adsk.eagle:package:23498/2"/>
 <part name="GND1" library="supply1" library_urn="urn:adsk.eagle:library:371" deviceset="GND" device=""/>
 <part name="GND2" library="supply1" library_urn="urn:adsk.eagle:library:371" deviceset="GND" device=""/>
-<part name="U$2" library="OPENBOT" library_urn="urn:adsk.eagle:library:760642" deviceset="CONN_02_PUI" device="XT60"/>
+<part name="U$2" library="OPENBOT" library_urn="urn:adsk.eagle:library:760642" deviceset="CONN_02_PUI" device="XT60" package3d_urn="urn:adsk.eagle:package:16508586/1"/>
 <part name="GND3" library="supply1" library_urn="urn:adsk.eagle:library:371" deviceset="GND" device=""/>
 <part name="R2" library="rcl" library_urn="urn:adsk.eagle:library:334" deviceset="R-EU_" device="0204/7" package3d_urn="urn:adsk.eagle:package:23498/2"/>
 <part name="D2" library="OPENBOT" library_urn="urn:adsk.eagle:library:760642" deviceset="LED" device="5MM" package3d_urn="urn:adsk.eagle:package:760648/2"/>
 <part name="GND4" library="supply1" library_urn="urn:adsk.eagle:library:371" deviceset="GND" device=""/>
-<part name="U$4" library="OPENBOT" library_urn="urn:adsk.eagle:library:760642" deviceset="CONN_02_PUI" device="XT60"/>
+<part name="U$4" library="OPENBOT" library_urn="urn:adsk.eagle:library:760642" deviceset="CONN_02_PUI" device="XT60" package3d_urn="urn:adsk.eagle:package:16508586/1"/>
 <part name="D3" library="OPENBOT" library_urn="urn:adsk.eagle:library:760642" deviceset="LED" device="5MM" package3d_urn="urn:adsk.eagle:package:760648/2"/>
 <part name="R3" library="rcl" library_urn="urn:adsk.eagle:library:334" deviceset="R-EU_" device="0204/7" package3d_urn="urn:adsk.eagle:package:23498/2"/>
 <part name="GND5" library="supply1" library_urn="urn:adsk.eagle:library:371" deviceset="GND" device=""/>
 <part name="GND6" library="supply1" library_urn="urn:adsk.eagle:library:371" deviceset="GND" device=""/>
-<part name="U$7" library="OPENBOT" library_urn="urn:adsk.eagle:library:760642" deviceset="CONN_02_PUI" device="XT60"/>
+<part name="U$7" library="OPENBOT" library_urn="urn:adsk.eagle:library:760642" deviceset="CONN_02_PUI" device="XT60" package3d_urn="urn:adsk.eagle:package:16508586/1"/>
 <part name="D4" library="OPENBOT" library_urn="urn:adsk.eagle:library:760642" deviceset="LED" device="5MM" package3d_urn="urn:adsk.eagle:package:760648/2"/>
 <part name="R4" library="rcl" library_urn="urn:adsk.eagle:library:334" deviceset="R-EU_" device="0204/7" package3d_urn="urn:adsk.eagle:package:23498/2"/>
 <part name="GND7" library="supply1" library_urn="urn:adsk.eagle:library:371" deviceset="GND" device=""/>
 <part name="GND8" library="supply1" library_urn="urn:adsk.eagle:library:371" deviceset="GND" device=""/>
-<part name="U$1" library="OPENBOT" library_urn="urn:adsk.eagle:library:760642" deviceset="AUTOMOTIVE_FUSE" device=""/>
-<part name="U$3" library="OPENBOT" library_urn="urn:adsk.eagle:library:760642" deviceset="AUTOMOTIVE_FUSE" device=""/>
-<part name="U$5" library="OPENBOT" library_urn="urn:adsk.eagle:library:760642" deviceset="AUTOMOTIVE_FUSE" device=""/>
+<part name="U$1" library="OPENBOT" library_urn="urn:adsk.eagle:library:760642" deviceset="AUTOMOTIVE_FUSE" device="" package3d_urn="urn:adsk.eagle:package:16508585/6"/>
+<part name="U$3" library="OPENBOT" library_urn="urn:adsk.eagle:library:760642" deviceset="AUTOMOTIVE_FUSE" device="" package3d_urn="urn:adsk.eagle:package:16508585/6"/>
+<part name="U$5" library="OPENBOT" library_urn="urn:adsk.eagle:library:760642" deviceset="AUTOMOTIVE_FUSE" device="" package3d_urn="urn:adsk.eagle:package:16508585/6"/>
 <part name="P+1" library="supply1" library_urn="urn:adsk.eagle:library:371" deviceset="+12V" device=""/>
+<part name="U$8" library="OPENBOT" library_urn="urn:adsk.eagle:library:760642" deviceset="CONN_02_PUI" device="XT60" package3d_urn="urn:adsk.eagle:package:16508586/1"/>
+<part name="D5" library="OPENBOT" library_urn="urn:adsk.eagle:library:760642" deviceset="LED" device="5MM" package3d_urn="urn:adsk.eagle:package:760648/2"/>
+<part name="R5" library="rcl" library_urn="urn:adsk.eagle:library:334" deviceset="R-EU_" device="0204/7" package3d_urn="urn:adsk.eagle:package:23498/2"/>
+<part name="GND9" library="supply1" library_urn="urn:adsk.eagle:library:371" deviceset="GND" device=""/>
+<part name="GND10" library="supply1" library_urn="urn:adsk.eagle:library:371" deviceset="GND" device=""/>
+<part name="U$9" library="OPENBOT" library_urn="urn:adsk.eagle:library:760642" deviceset="AUTOMOTIVE_FUSE" device="" package3d_urn="urn:adsk.eagle:package:16508585/6"/>
 </parts>
 <sheets>
@@
 <attribute name="VALUE" x="54.61" y="69.85" size="1.778" layer="96" rot="R90"/>
 </instance>
+<instance part="U$8" gate="G$1" x="10.16" y="6.35" smashed="yes" rot="MR0">
+<attribute name="NAME" x="12.7" y="8.89" size="1.778" layer="95" rot="MR0"/>
+</instance>
+<instance part="D5" gate="G$1" x="21.59" y="-8.89" smashed="yes">
+<attribute name="NAME" x="18.288" y="-8.001" size="1.778" layer="95" font="vector"/>
+<attribute name="VALUE" x="23.495" y="-13.462" size="1.778" layer="96" font="vector" rot="R90" align="top-left"/>
+</instance>
+<instance part="R5" gate="G$1" x="21.59" y="0" smashed="yes" rot="R90">
+<attribute name="NAME" x="17.78" y="2.7686" size="1.778" layer="95"/>
+<attribute name="VALUE" x="24.892" y="-3.81" size="1.778" layer="96" rot="R90"/>
+</instance>
+<instance part="GND9" gate="1" x="16.51" y="0" smashed="yes">
+<attribute name="VALUE" x="13.97" y="-2.54" size="1.778" layer="96"/>
+</instance>
+<instance part="GND10" gate="1" x="21.59" y="-17.78" smashed="yes">
+<attribute name="VALUE" x="19.05" y="-20.32" size="1.778" layer="96"/>
+</instance>
+<instance part="U$9" gate="G$1" x="30.48" y="6.35" smashed="yes"/>
 </instances>
 <busses>
@@
 <pinref part="D4" gate="G$1" pin="C"/>
 <wire x1="21.59" y1="77.47" x2="21.59" y2="78.74" width="0.1524" layer="91"/>
+</segment>
+<segment>
+<pinref part="GND9" gate="1" pin="GND"/>
+<pinref part="U$8" gate="G$1" pin="GND/COM"/>
+<wire x1="16.51" y1="2.54" x2="16.51" y2="3.81" width="0.1524" layer="91"/>
+<wire x1="16.51" y1="3.81" x2="14.605" y2="3.81" width="0.1524" layer="91"/>
+</segment>
+<segment>
+<pinref part="GND10" gate="1" pin="GND"/>
+<pinref part="D5" gate="G$1" pin="C"/>
+<wire x1="21.59" y1="-15.24" x2="21.59" y2="-13.97" width="0.1524" layer="91"/>
 </segment>
 </net>
@@
 <junction x="57.15" y="68.58"/>
 <wire x1="38.1" y1="36.83" x2="43.18" y2="36.83" width="0.1524" layer="91"/>
-<wire x1="43.18" y1="36.83" x2="43.18" y2="68.58" width="0.1524" layer="91"/>
+<wire x1="43.18" y1="36.83" x2="43.18" y2="38.1" width="0.1524" layer="91"/>
 <junction x="43.18" y="68.58"/>
+<wire x1="43.18" y1="38.1" x2="43.18" y2="68.58" width="0.1524" layer="91"/>
 <wire x1="38.1" y1="99.06" x2="43.18" y2="99.06" width="0.1524" layer="91"/>
 <wire x1="43.18" y1="99.06" x2="43.18" y2="68.58" width="0.1524" layer="91"/>
@@
 <pinref part="P+1" gate="1" pin="+12V"/>
 <wire x1="57.15" y1="72.39" x2="57.15" y2="68.58" width="0.1524" layer="91"/>
+<pinref part="U$9" gate="G$1" pin="P$1"/>
+<wire x1="38.1" y1="6.35" x2="43.18" y2="6.35" width="0.1524" layer="91"/>
+<wire x1="43.18" y1="6.35" x2="43.18" y2="36.83" width="0.1524" layer="91"/>
+</segment>
+</net>
+<net name="N$3" class="0">
+<segment>
+<pinref part="U$8" gate="G$1" pin="V+/VCC"/>
+<wire x1="14.605" y1="6.35" x2="21.59" y2="6.35" width="0.1524" layer="91"/>
+<pinref part="R5" gate="G$1" pin="2"/>
+<wire x1="21.59" y1="6.35" x2="22.86" y2="6.35" width="0.1524" layer="91"/>
+<wire x1="21.59" y1="5.08" x2="21.59" y2="6.35" width="0.1524" layer="91"/>
+<junction x="21.59" y="6.35"/>
+<pinref part="U$9" gate="G$1" pin="P$2"/>
+</segment>
+</net>
+<net name="N$9" class="0">
+<segment>
+<pinref part="D5" gate="G$1" pin="A"/>
+<pinref part="R5" gate="G$1" pin="1"/>
+<wire x1="21.59" y1="-6.35" x2="21.59" y2="-5.08" width="0.1524" layer="91"/>
 </segment>
 </net>
@@
 for full support of SPICE simulation.
 </note>
+<note version="8.5" severity="warning">
+Since Version 8.5, EAGLE supports locking for holes, vias, wires and polygons.
+The locking property on all objects of these types will not be understood in this version.
+</note>
 </compatibility>
