File: 01 - CDRF/01 - ELECTRONIQUE/CAPTEUR_HALL/AdaptSensor.brd (EAGLE design)
At the start: 17.6 x 14.4 mm, 5 parts

Commit message: update pcb
Parts:
- flipped J1 to the bottom
Changed lines of the file:
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@@
 </layers>
 <board>
+<fusionsync huburn="a.cGVyc29uYWw6dWUyOGY1Yzgw" projecturn="a.cGVyc29uYWw6dWUyOGY1YzgwIzIwMTgwNTEzMTMxNzkwNTU2" f3durn="urn:adsk.wipprod:dm.lineage:X1HgFxsWRoqEliTZEj40CQ" pcbguid="e07dd0c2-51ef-48ca-b847-8229884f9b68" lastpulledtime="" lastsyncedchangeguid="e5276c8e-fbce-6b2c-9c3c-80e73cf65c6e"/>
 <plain>
 <wire x1="0" y1="0" x2="17.633" y2="0" width="0" layer="20"/>
@@
 <attribute name="VALUE" x="6.056709375" y="7.867490625" size="1.272140625" layer="27" rot="R90"/>
 </element>
-<element name="J1" library="CONNECTORS" library_urn="urn:adsk.eagle:library:786230" package="MOLEX-1X3" package3d_urn="urn:adsk.eagle:package:786243/2" value="" x="9.398" y="5.969" smashed="yes" rot="R90">
-<attribute name="NAME" x="7.239" y="7.112" size="0.6096" layer="25" font="vector" ratio="20" rot="R90"/>
-<attribute name="PROD_ID" value="CONN-08625" x="20.828" y="26.289" size="1.778" layer="27" rot="R90" display="off"/>
-<attribute name="SF_ID" value="PRT-08096" x="20.828" y="26.289" size="1.778" layer="27" rot="R90" display="off"/>
-<attribute name="VALUE" x="8.128" y="6.858" size="0.6096" layer="27" font="vector" ratio="20" rot="R90"/>
+<element name="J1" library="CONNECTORS" library_urn="urn:adsk.eagle:library:786230" package="MOLEX-1X3" package3d_urn="urn:adsk.eagle:package:786243/2" value="" x="9.398" y="5.969" smashed="yes" rot="MR90">
+<attribute name="NAME" x="11.557" y="7.112" size="0.6096" layer="26" font="vector" ratio="20" rot="MR90"/>
+<attribute name="PROD_ID" value="CONN-08625" x="-2.032" y="26.289" size="1.778" layer="28" rot="MR90" display="off"/>
+<attribute name="SF_ID" value="PRT-08096" x="-2.032" y="26.289" size="1.778" layer="28" rot="MR90" display="off"/>
+<attribute name="VALUE" x="10.668" y="6.858" size="0.6096" layer="28" font="vector" ratio="20" rot="MR90"/>
 </element>
 <element name="R1" library="fab" library_urn="urn:adsk.eagle:library:9340542" package="R1206FAB" package3d_urn="urn:adsk.eagle:package:9340722/2" value="" x="4.064" y="4.191" smashed="yes" rot="R90">
@@
 <contactref element="U$1" pad="2"/>
 <wire x1="9.525" y1="2.54" x2="9.525" y2="5.842" width="0.8128" layer="1"/>
-<wire x1="9.525" y1="5.842" x2="9.398" y2="5.969" width="0.8128" layer="1"/>
-<wire x1="9.398" y1="5.969" x2="13.462" y2="5.969" width="0.8128" layer="1"/>
 <wire x1="1.77858125" y1="9.779" x2="1.77858125" y2="11.30358125" width="0.8128" layer="1"/>
 <wire x1="1.77858125" y1="11.30358125" x2="3.429" y2="12.954" width="0.8128" layer="1"/>
@@
 <wire x1="16.129" y1="6.604" x2="15.494" y2="5.969" width="0.8128" layer="1"/>
 <wire x1="15.494" y1="5.969" x2="13.462" y2="5.969" width="0.8128" layer="1"/>
+<wire x1="9.398" y1="5.969" x2="13.462" y2="5.969" width="0.8128" layer="1"/>
+<wire x1="9.398" y1="5.969" x2="9.525" y2="5.842" width="0" layer="19" extent="1-1"/>
 </signal>
 <signal name="+5V">
@@
 <contactref element="R1" pad="2"/>
 <contactref element="C1" pad="1"/>
-<wire x1="3.981" y1="8.829" x2="9.078" y2="8.829" width="0.8128" layer="1"/>
-<wire x1="9.078" y1="8.829" x2="9.398" y2="8.509" width="0.8128" layer="1"/>
-<wire x1="9.398" y1="8.509" x2="10.16" y2="9.271" width="0.8128" layer="1"/>
-<wire x1="10.16" y1="9.271" x2="13.462" y2="9.271" width="0.8128" layer="1"/>
+<wire x1="13.462" y1="9.271" x2="10.16" y2="9.271" width="0.8128" layer="1"/>
 <wire x1="4.064" y1="5.842" x2="4.064" y2="8.746" width="0.8128" layer="1"/>
 <wire x1="4.064" y1="8.746" x2="3.981" y2="8.829" width="0.8128" layer="1"/>
+<wire x1="9.078" y1="8.829" x2="9.398" y2="8.509" width="0.8128" layer="1"/>
+<wire x1="3.981" y1="8.829" x2="9.078" y2="8.829" width="0.8128" layer="1"/>
+<wire x1="10.16" y1="9.271" x2="9.398" y2="8.509" width="0.8128" layer="1"/>
 </signal>
 <signal name="CAPT">
 <contactref element="J1" pad="3"/>
 <contactref element="D1" pad="2"/>
-<wire x1="3.981" y1="10.729" x2="9.078" y2="10.729" width="0.8128" layer="1"/>
-<wire x1="9.078" y1="10.729" x2="9.398" y2="11.049" width="0.8128" layer="1"/>
+<wire x1="9.078" y1="10.729" x2="3.981" y2="10.729" width="0.8128" layer="1"/>
+<wire x1="9.398" y1="11.049" x2="9.078" y2="10.729" width="0.8128" layer="1"/>
 </signal>
 <signal name="N$1">
@@
 </note>
 <note version="8.3" severity="warning">
+Since Version 8.3, EAGLE supports Fusion synchronisation.
+This feature will not be available in this version and saving
+the document will break the link to the Fusion PCB feature.
+</note>
+<note version="8.3" severity="warning">
