File: 01 - CDRF/01 - ELECTRONIQUE/MAIN_BOARD V2/MAIN_BOARD_02.sch (EAGLE design)
At the start: 39 parts, among them J5 CONN_05, J6 CONN_05, J8 CONN_05, U1 74HC165SO-16

Commit message: update PCB
Parts:
- removed C9: 100uF, rcl:CPOL-EUE5-10.5
- added C1, C2: 10uF, rcl:CPOL-EU153CLV-0505
Connections:
- net +5V: now also C2.+; no longer C9.+
- net GND: now also C1.-, C2.-; no longer C9.-
- net IO-ADVERSAIRE1: now also U$1.33/T
- net IO-ADVERSAIRE2: now also U$1.32/T/PWM
- net IO-BORDURE1: now also U$1.17/A3/T; no longer U$1.16/A2/T
- net IO-BORDURE2: now also U$1.16/A2/T; no longer U$1.15/A1/T
- net IO-BORDURE3: now also U$1.15/A1/T; no longer U$1.14/A0
- net IO-BORDURE4: now also U$1.14/A0
- net VIN/BATT: now also C1.+
Other:
- note added: "C1 et C2 Ref GoTronic : 22438"
- moved on the sheet: LED4, R10

Commit message: Update PCB
Parts:
- added U$3, U$4: LOGO_K, KARIBOUS:LOGO_K
Connections:
- net MISO_DRIVER: now also J8.1; no longer J8.2
- net SCK_DRIVER: now also J8.2; no longer J8.1
Other:
- moved on the sheet: J1, J2, J3, J4, J7, J8, R3, R4, U$1, U$2

Commit message: update PCB
Parts:
- removed R10: (no value), rcl:R-EU_R1206
- added P1: 10k, rcl:POTENTIOMETER_PT-10
- R2: value 10k -> (none); device rcl:POTENTIOMETER_PT-10 -> rcl:R-EU_R1206
- renumbered COM-XBEE1 to COM-BALISE, J1 to CON-SAT3, J10 to CON-LCD, J2 to CON-SAT2, J3 to CON-SAT1, J4 to CON-SAT4, J5 to ENCODEUR_GAUCHE, J6 to ENCODEUR_DROIT, J7 to DRIVER-MOTEUR, J8 to SPI-DRIVER, J9 to CON-IHM, LED1 to LED_REGUL, LED4 to LED_BATT, R7 to R5, RN3 to RN1
Connections:
- net +3V3/1: now also R2.2; no longer R4.2
- net +5V: now also P1.2; no longer R2.2
- net GND: now also P1.1; no longer R2.1
- net LCD_V0: now also P1.3; no longer R2.3
- net N$3: now also R4.1; no longer R10.1
- net SCL: now also R2.1; no longer R4.1
- net VIN/BATT: now also R4.2; no longer R10.2
