File: 01 - CDRF/01 - ELECTRONIQUE/MAIN_BOARD V2/MAIN_BOARD_02.brd (EAGLE design)
At the start: 85 x 85 mm, 39 parts, among them J5 CONN_05, J6 CONN_05, J8 CONN_05, U1 74HC165SO-16

Commit message: update PCB
Parts:
- removed C9: 100uF, rcl:E5-10,5
- added C1, C2: 10uF, rcl:153CLV-0505
- moved ADVERSAIRE_2 19.7 mm to (24.8, 2.54)
- moved ALIM_OUT1 19.7 mm to (16.5, 12.1), turned to 90 degrees
- moved ADVERSAIRE_1 19.4 mm to (31.8, 2.54)
- moved D1 16.6 mm to (4.83, 24.4), flipped to the bottom, turned to 270 degrees
- moved R1 14.5 mm to (1.91, 60.3), turned to 90 degrees
- moved PS1 12.0 mm to (5.71, 24.4), turned to 270 degrees
- moved R10 11.9 mm to (9.53, 11.4)
- moved LED4 11.7 mm to (3.81, 11.4)
- moved COM-XBEE 8.28 mm to (17.1, 45.7), turned to 90 degrees
- moved BORDURE_4 7.85 mm to (38.7, 2.54)
- moved BORDURE_1 7.85 mm to (59.7, 2.54)
- moved BORDURE_2 7.85 mm to (52.7, 2.54)
- moved BORDURE_3 7.85 mm to (45.7, 2.54)
- moved R7 4.96 mm to (9.53, 15.2)
- moved LED1 4.58 mm to (3.81, 15.2)
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Connections:
- net +5V: now also C2.+; no longer C9.+
- net GND: now also C1.-, C2.-; no longer C9.-
- net IO-ADVERSAIRE1: now also U$1.33
- net IO-ADVERSAIRE2: now also U$1.32
- net IO-BORDURE1: now also U$1.17/A3; no longer U$1.16/A2
- net IO-BORDURE2: now also U$1.16/A2; no longer U$1.15/A1
- net IO-BORDURE3: now also U$1.15/A1; no longer U$1.14/A0
- net IO-BORDURE4: now also U$1.14/A0
- net VIN/BATT: now also C1.+

Commit message: Update PCB
Parts:
- added U$3, U$4: LOGO_K, KARIBOUS:LOGO_KARIBOU
- moved R1 12.0 mm to (5.71, 48.9), turned to 0 degrees
- moved ALIM_OUT1 9.61 mm to (17.8, 2.54)
- moved R3 4.64 mm to (75.4, 46.2)
- moved LED4 4.45 mm to (3.81, 15.9)
- moved R10 4.45 mm to (9.53, 15.9)
- moved LED1 3.18 mm to (3.81, 12.1)
- moved R7 3.18 mm to (9.53, 12.1)
- moved RN2 2.69 mm to (38.7, 43.8)
- moved R4 2.05 mm to (75.4, 49.5)
- moved J9 2.01 mm to (31.1, 31.8)
- moved U1 2.01 mm to (31.1, 43.8)
- moved C2 1.91 mm to (14.6, 22.2)
- moved RN3 1.91 mm to (24.1, 43.8)
- moved J8 1.27 mm to (50.2, 35.6)
- moved C1 1.27 mm to (14.6, 29.8)
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Connections:
- net MISO_DRIVER: now also J8.1; no longer J8.2
- net SCK_DRIVER: now also J8.2; no longer J8.1
Routing:
- net +5V: track 0.00 -> 253.0 mm
- net SCL: track 0.00 -> 95.9 mm
- net SDA: track 0.00 -> 86.9 mm
- net +3V3/1: track 0.00 -> 75.9 mm
- net MISO: track 0.00 -> 64.9 mm
- net SCK: track 0.00 -> 56.8 mm
- net MOSI: track 0.00 -> 51.2 mm
- net IO-ADVERSAIRE2: track 0.00 -> 41.8 mm
- net VIN/BATT: track 0.00 -> 39.9 mm
- net IO-ADVERSAIRE1: track 0.00 -> 38.1 mm
- net CON3-7: track 0.00 -> 33.2 mm
- net CON3-8: track 0.00 -> 31.4 mm
- net D3: track 0.00 -> 30.9 mm
- net D4: track 0.00 -> 30.0 mm
- net M0: track 0.00 -> 28.6 mm
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- added copper zone on layer 1, net GND
- added copper zone on layer 16, net GND

Commit message: update PCB
Parts:
- removed R10: (no value), rcl:R1206
- added P1: 10k, rcl:PT-10
- R2: value 10k -> (none); device rcl:PT-10 -> rcl:R1206
- moved R4 74.0 mm to (9.53, 15.9)
- moved R2 61.0 mm to (75.4, 49.5), turned to 0 degrees
- moved U$4 8.98 mm to (45.7, 11.4)
- moved U$3 5.85 mm to (19.7, 11.4)
- renumbered COM-XBEE1 to COM-BALISE, J1 to CON-SAT3, J10 to CON-LCD, J2 to CON-SAT2, J3 to CON-SAT1, J4 to CON-SAT4, J5 to ENCODEUR_GAUCHE, J6 to ENCODEUR_DROIT, J7 to DRIVER-MOTEUR, J8 to SPI-DRIVER, J9 to CON-IHM, LED1 to LED_REGUL, LED4 to LED_BATT, R7 to R5, RN3 to RN1
Connections:
- net +3V3/1: now also R2.2; no longer R4.2
- net +5V: now also P1.2; no longer R2.2
- net GND: now also P1.1; no longer R2.1
- net LCD_V0: now also P1.3; no longer R2.3
- net N$3: now also R4.1; no longer R10.1
- net SCL: now also R2.1; no longer R4.1
- net VIN/BATT: now also R4.2; no longer R10.2
Other:
- board text added: "MAIN-BOARD V2 2020 Barbatronic cc-by"
