File: 01 - CDRF/01 - ELECTRONIQUE/PCB_BALISE_328P/PCB_BALISE_328P.sch (EAGLE design)
At the start: 16 parts

Commit message: electrical update
Parts:
- removed ADC_1, DIGITAL_2, POWER: (no value), pinhead:PINHD-1X2
- removed ADC_2: (no value), con-lstb:MA04-1
- removed C2: 22pF, AVX_By_element14_Batch_1:0612ZC225MAT2A
- removed C5: 100nF, 01_SparkFun:CAP1206
- removed D13: M01PTH, 01_SparkFun:M01PTH
- removed DIGITAL1: (no value), con-lstb:MA03-1
- removed DIGITAL_3: (no value), con-lstb:MA08-1
- added C6, C7: 0,1uF, rcl:C-EUC1206K
- added C8: 22pF, rcl:C-EUC1206K
- added D1: M7, fab:CDBM1100-G
- added D2: GF1, diode:GF1
- added J1: (no value), OPENBOT:CONN_04POLAR
- added J2: (no value), OPENBOT:CONN_02POLAR
- added LED1: (no value), led:LEDSMT1206
- added LED_BATT, LED_REGUL: (no value), eagle-ltspice:LED_E
- added PS2: R-78B5.0-2.0, OPENBOT:R-78B5.0-2.0
- added R2, R5, R6: (no value), rcl:R-EU_R1206
- added R3, R4: 1k, rcl:R-EU_R1206
- added R7: 10k, rcl:R-EU_R1206
- added R8: 1K, rcl:R-EU_R1206
- added RU1: RUEF300, OPENBOT:RUEF300
- added T1: (no value), fab:NMOSFETSOT23
- added U$5: CONN_02_PUIXT30, OPENBOT:CONN_02_PUIXT30
- C1: device AVX_By_element14_Batch_1:0612ZC225MAT2A -> rcl:C-EUC1206K
- C3: device 01_SparkFun:CAP1206 -> rcl:CPOL-EU153CLV-0505
- C4: value 1uF -> 10uF; device 01_SparkFun:CAP1206 -> rcl:CPOL-EU153CLV-0505
- R1: value 10k -> 1K; device 01_SparkFun:RESISTOR1206 -> rcl:R-EU_R1206
Connections:
- removed net ADC0: ADC_1.1, MICRO.PC0(ADC0/PCINT8)
- removed net ADC1: ADC_1.2, MICRO.PC1(ADC1/PCINT9)
- removed net ADC2: ADC_2.1, MICRO.PC2(ADC2/PCINT10)
- removed net ADC3: ADC_2.2, MICRO.PC3(ADC3/PCINT11)
- removed net ADC4/SDA: ADC_2.3, MICRO.PC4(ADC4/SDA/PCINT12)
- removed net ADC5/SCL: ADC_2.4, MICRO.PC5(ADC5/SCL/PCINT13)
- removed net D0/TX: DIGITAL1.1, MICRO.PD0(RXD/PCINT16)
- removed net D1/RX: DIGITAL1.2, MICRO.PD1(TXD/PCINT17)
- removed net D10: DIGITAL_3.6, MICRO.PB2(SS/OC1B/PCINT2)
- removed net D11: DIGITAL_3.7, MICRO.PB3(MOSI/OC2A/PCINT3)
- removed net D12: DIGITAL_3.8, MICRO.PB4(MISO/PCINT4)
- removed net D13: D13.1, MICRO.PB5(SCK/PCINT5)
- removed net D2: DIGITAL1.3, MICRO.PD2(INT0/PCINT18)
- removed net D3: DIGITAL_2.1, MICRO.PD3(INT1/OC2B/PCINT19)
- removed net D4: DIGITAL_2.2, MICRO.PD4(T0/XCK/PCINT20)
- removed net D5: DIGITAL_3.1, MICRO.PD5(T1/OC0B/PCINT21)
- removed net D6: DIGITAL_3.2, MICRO.PD6(AIN0/OC0A/PCINT22)
- removed net D7: DIGITAL_3.3, MICRO.PD7(AIN1/PCINT23)
- removed net D8: DIGITAL_3.4, MICRO.PB0(ICP1/CLKO/PCINT0)
- removed net D9: DIGITAL_3.5, MICRO.PB1(OC1A/PCINT1)
- removed net VCC: C3.1, C4.1, C5.1, MICRO.AREF, MICRO.AVCC, MICRO.VCC@1, MICRO.VCC@2, POWER.2, R1.1, U$1.VCC
- new net +5V: C4.+, C6.1, D1.ANODE, D2.C, J2.1, MICRO.AVCC, MICRO.VCC@1, MICRO.VCC@2, PS2.+VOUT, R1.2, R5.2, U$1.VCC
- new net N$1: C7.1, MICRO.AREF
- new net N$10: LED_REGUL.A, R5.1
- new net N$11: D2.A, J2.2, T1.D
- new net N$12: R7.2, R8.2, T1.G
- new net N$3: LED1.A, R2.1
- new net N$4: MICRO.PD0(RXD/PCINT16), R3.2
- new net N$5: MICRO.PD1(TXD/PCINT17), R4.2
- new net N$6: J1.2, MICRO.PD2(INT0/PCINT18)
- new net N$7: LED_BATT.A, R6.1
- new net N$8: RU1.P$1, U$5.V+/VCC
- new net PUMP: R8.1
- new net RX: J1.3, R4.1
- new net TX: J1.4, R3.1
- new net VIN/BATT: C3.+, D1.KATHODE, PS2.+VIN, R6.2, RU1.P$2
- net GND: now also C1.1, C3.-, C4.-, C6.2, C7.2, C8.1, J1.1, LED1.C, LED_BATT.C, LED_REGUL.C, PS2.GND, R7.1, T1.S, U$5.GND/COM; no longer C1.C1, C2.C1, C3.2, C4.2, C5.2, POWER.1
- net MISO: now also MICRO.PB4(MISO/PCINT4)
- net MOSI: now also MICRO.PB3(MOSI/OC2A/PCINT3)
- net N$2: now also C8.2; no longer C1.C2
- net N$9: now also C1.2; no longer C2.C2
- net RST: now also R1.1; no longer R1.2
- net SCK: now also MICRO.PB5(SCK/PCINT5), R2.2
Other:
- note added: "C1 et C2 Ref GoTronic : 22438"
- moved on the sheet: CRYSTAL, MICRO, U$1
