File: 01 - CDRF/01 - ELECTRONIQUE/PCB_BALISE_328P/PCB_BALISE_328P.brd (EAGLE design)
At the start: 38.9 x 28.3 mm, 16 parts

Commit message: electrical update
Parts:
- removed ADC_1, DIGITAL_2, POWER: (no value), pinhead:1X02
- removed ADC_2: (no value), con-lstb:MA04-1
- removed C2: 22pF, AVX_By_element14_Batch_1:CAPC3216X178N
- removed C5: 100nF, 01_SparkFun:1206
- removed D13: M01PTH, 01_SparkFun:1X01
- removed DIGITAL1: (no value), con-lstb:MA03-1
- removed DIGITAL_3: (no value), con-lstb:MA08-1
- added C6, C7: 0,1uF, rcl:C1206K
- added C8: 22pF, rcl:C1206K
- added D1: M7, fab:MINI-SMA
- added D2: GF1, diode:SMA-DO214AC
- added J1: (no value), OPENBOT:MOLEX-1X4
- added J2: (no value), OPENBOT:MOLEX-1X2
- added LED1: (no value), led:1206
- added LED_BATT, LED_REGUL: (no value), eagle-ltspice:LED_1206
- added PS2: R-78B5.0-2.0, OPENBOT:CONV_R-78B5.0-2.0
- added R2, R5, R6: (no value), rcl:R1206
- added R3, R4: 1k, rcl:R1206
- added R7: 10k, rcl:R1206
- added R8: 1K, rcl:R1206
- added RU1: RUEF300, OPENBOT:RUEF300
- added T1: (no value), fab:SOT-23
- added U$5: CONN_02_PUIXT30, OPENBOT:XT30_FEMALE
- C1: device AVX_By_element14_Batch_1:CAPC3216X178N -> rcl:C1206K
- C3: device 01_SparkFun:1206 -> rcl:153CLV-0505
- C4: value 1uF -> 10uF; device 01_SparkFun:1206 -> rcl:153CLV-0505
- R1: value 10k -> 1K; device 01_SparkFun:1206 -> rcl:R1206
- moved U$1 71.6 mm to (29.1, 68.4)
- moved C3 56.0 mm to (16.5, 68.6), turned to 0 degrees
- moved C1 47.2 mm to (26.7, 49.5), turned to 0 degrees
- moved C4 46.3 mm to (3.81, 53.3), turned to 0 degrees
- moved R1 33.9 mm to (26.7, 43.2), turned to 0 degrees
Connections:
- removed net ADC0: ADC_1.1, MICRO.23
- removed net ADC1: ADC_1.2, MICRO.24
- removed net ADC2: ADC_2.1, MICRO.25
- removed net ADC3: ADC_2.2, MICRO.26
- removed net ADC4/SDA: ADC_2.3, MICRO.27
- removed net ADC5/SCL: ADC_2.4, MICRO.28
- removed net D0/TX: DIGITAL1.1, MICRO.30
- removed net D1/RX: DIGITAL1.2, MICRO.31
- removed net D10: DIGITAL_3.6, MICRO.14
- removed net D11: DIGITAL_3.7, MICRO.15
- removed net D12: DIGITAL_3.8, MICRO.16
- removed net D13: D13.1, MICRO.17
- removed net D2: DIGITAL1.3, MICRO.32
- removed net D3: DIGITAL_2.1, MICRO.1
- removed net D4: DIGITAL_2.2, MICRO.2
- removed net D5: DIGITAL_3.1, MICRO.9
- removed net D6: DIGITAL_3.2, MICRO.10
- removed net D7: DIGITAL_3.3, MICRO.11
- removed net D8: DIGITAL_3.4, MICRO.12
- removed net D9: DIGITAL_3.5, MICRO.13
- removed net VCC: C3.1, C4.1, C5.1, MICRO.18, MICRO.20, MICRO.4, MICRO.6, POWER.2, R1.1, U$1.2
- new net +5V: C4.+, C6.1, D1.ANODE, D2.K, J2.1, MICRO.18, MICRO.4, MICRO.6, PS2.3, R1.2, R5.2, U$1.2
- new net N$1: C7.1, MICRO.20
- new net N$10: LED_REGUL.A, R5.1
- new net N$11: D2.A, J2.2, T1.1
- new net N$12: R7.2, R8.2, T1.3
- new net N$3: LED1.A, R2.1
- new net N$4: MICRO.30, R3.2
- new net N$5: MICRO.31, R4.2
- new net N$6: J1.2, MICRO.32
- new net N$7: LED_BATT.A, R6.1
- new net N$8: RU1.P$1, U$5.P$1
- new net PUMP: R8.1
- new net RX: J1.3, R4.1
- new net TX: J1.4, R3.1
- new net VIN/BATT: C3.+, D1.KATHODE, PS2.1, R6.2, RU1.P$2
- net GND: now also C3.-, C4.-, C6.2, C7.2, C8.1, J1.1, LED1.C, LED_BATT.C, LED_REGUL.C, PS2.2, R7.1, T1.2, U$5.P$2; no longer C2.1, C3.2, C4.2, C5.2, POWER.1
- net MISO: now also MICRO.16
- net MOSI: now also MICRO.15
- net N$2: now also C8.2; no longer C1.2
- net N$9: now also C1.2; no longer C2.2
- net RST: now also R1.1; no longer R1.2
- net SCK: now also MICRO.17, R2.2
Routing:
- net RST: track 28.7 -> 0.00 mm
- net VCC: track 24.4 -> 0.00 mm
- net N$2: track 19.0 -> 1.24 mm
- net D2: track 16.8 -> 0.00 mm
- net D1/RX: track 15.4 -> 0.00 mm
- net D12: track 14.4 -> 0.00 mm
- net GND: track 13.3 -> 0.00 mm
- net ADC2: track 13.0 -> 0.00 mm
- net D11: track 12.6 -> 0.00 mm
- net D10: track 12.1 -> 0.00 mm
- net D0/TX: track 12.1 -> 0.00 mm
- net ADC3: track 11.5 -> 0.00 mm
- net D3: track 11.2 -> 0.00 mm
- net D9: track 10.7 -> 0.00 mm
- net N$9: track 12.0 -> 1.62 mm
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
Commit message: cleanup
Parts:
- added C2, C5: (no value), rcl:C1206K
- added IC1: (no value), fab:SOT23
- added J3, J4: (no value), OPENBOT:MOLEX-1X4
- added J5: (no value), OPENBOT:MOLEX-1X3
- added R10, R9: (no value), rcl:R1206
- added SPI_OLED: (no value), pinhead:1X07
- added U1: AVRISP, fab:2X03
- added U2: XBP24CAUIT-001, OPENBOT:MODULE_XBP24CAUIT-001
- U$1: value AVRISP -> LOGO_K; device fab:2X03 -> KARIBOUS:LOGO_KARIBOU
- moved U$1 91.4 mm to (19.0, -22.4)
- moved LED1 88.4 mm to (-20.3, -41.9), turned to 270 degrees
- moved R2 88.4 mm to (-20.3, -36.8), turned to 90 degrees
- moved PS2 87.3 mm to (-6.35, -20.3), turned to 270 degrees
- moved C3 87.3 mm to (-15.2, -12.7)
- moved LED_BATT 84.7 mm to (-12.7, -41.9), turned to 270 degrees
- moved C4 83.5 mm to (-15.2, -27.9)
- moved LED_REGUL 82.2 mm to (-16.5, -41.9), turned to 270 degrees
- moved RU1 77.1 mm to (2.54, -20.3), turned to 90 degrees
- moved R6 72.7 mm to (-12.7, -36.8), turned to 90 degrees
- moved R5 72.4 mm to (-16.5, -36.8), turned to 90 degrees
- moved C6 68.7 mm to (-15.9, 6.44)
- moved D1 66.8 mm to (-12.7, -20.3), turned to 270 degrees
- moved U$5 66.2 mm to (8.89, -20.3), turned to 90 degrees
- moved C7 63.7 mm to (-15.9, 9.13)
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Connections:
- removed net N$5: MICRO.31, R4.2
- removed net PUMP: R8.1
- new net CAPT_1: J3.4, MICRO.23
- new net CAPT_2: J3.3, MICRO.24
- new net CAPT_3: J4.4, MICRO.25
- new net CAPT_4: J4.3, MICRO.26
- new net CS: MICRO.14, SPI_OLED.7
- new net DC: MICRO.13, SPI_OLED.6
- new net HALL_SENSOR: J5.3, MICRO.27
- new net N$13: MICRO.1, R8.1
- new net N$15: R10.1, R9.1, U2.3
- new net RES: MICRO.12, SPI_OLED.5
- new net RX_RAW: MICRO.31, R4.2, U2.2
- new net TX_RAW: MICRO.30, R3.2, R9.2
- new net VREF: U2.14
- net +5V: now also C5.2, IC1.2, J3.2, J4.2, J5.2, SPI_OLED.2, U1.2; no longer U$1.2
- net GND: now also C2.1, C5.1, IC1.3, J3.1, J4.1, J5.1, R10.2, SPI_OLED.1, U1.6, U2.10; no longer U$1.6
- net MISO: now also U1.1; no longer U$1.1
- net MOSI: now also SPI_OLED.4, U1.4; no longer U$1.4
- net N$4: now also C2.2, IC1.1, U2.1; no longer MICRO.30, R3.2
- net RST: now also U1.5; no longer U$1.5
- net SCK: now also SPI_OLED.3, U1.3; no longer U$1.3
Routing:
- net +5V: track 0.00 -> 248.4 mm, vias 0 -> 1
- net N$13: track 0.00 -> 102.0 mm, vias 0 -> 2
- net SCK: track 0.00 -> 75.8 mm, vias 0 -> 1
- net TX_RAW: track 0.00 -> 62.7 mm
- net MOSI: track 0.00 -> 56.1 mm, vias 0 -> 1
- net RX_RAW: track 0.00 -> 55.2 mm
- net RES: track 0.00 -> 47.0 mm, vias 0 -> 1
- net VIN/BATT: track 0.00 -> 46.7 mm
- net DC: track 0.00 -> 44.5 mm, vias 0 -> 1
- net CS: track 0.00 -> 41.9 mm, vias 0 -> 1
- net HALL_SENSOR: track 0.00 -> 34.0 mm
- net N$6: track 0.00 -> 24.0 mm
- net CAPT_2: track 0.00 -> 18.7 mm
- net RST: track 0.00 -> 18.2 mm, vias 0 -> 2
- net CAPT_4: track 0.00 -> 17.6 mm
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- added copper zone on layer 1, net GND
- added copper zone on layer 16, net GND
Other:
- board size 38.9 x 28.3 mm -> 66 x 90.7 mm
- board text added: "+5V"
- board text added: "CS"
- board text added: "DC"
- board text added: "GND"
- board text added: "MOSI"
- board text added: "RES"
- board text added: "SCK"
