File: 01 - CDRF/01 - ELECTRONIQUE/PUMP PCB/PCB PUMP ATTINY.sch (EAGLE design)
At the start: 15 parts, among them IC1 ATTINY402-SSN, J3 PWRPAD2-5MM, J4 PWRPAD2-5MM

Commit message: add cap and led
Parts:
- added C2: (no value), rcl:CPOL-EU153CLV-0505
- added R5: 1K, rcl:R-EU_R1206
- added U$1: LEDFAB1206, fab:LEDFAB1206
Connections:
- new net N$6: R5.1, U$1.A
- new net N$7: IC1G$1.(LUT0-IN1/TCA0WO1/SDA/MOSI/AIN1)PA1, R5.2
- net +5V: now also C2.+
- net GND: now also C2.-, U$1.C
Changed lines of the file:
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@@
 <part name="C1" library="rcl" library_urn="urn:adsk.eagle:library:334" deviceset="C-EU" device="C1206" package3d_urn="urn:adsk.eagle:package:23618/2"/>
 <part name="JP3" library="pinhead-2" library_urn="urn:adsk.eagle:library:22357987" deviceset="PINHD-1X01" device="_2.54-SMD" package3d_urn="urn:adsk.eagle:package:22358666/1"/>
+<part name="C2" library="rcl" library_urn="urn:adsk.eagle:library:334" deviceset="CPOL-EU" device="153CLV-0505" package3d_urn="urn:adsk.eagle:package:23402/2"/>
+<part name="GND7" library="supply1" library_urn="urn:adsk.eagle:library:371" deviceset="GND" device=""/>
+<part name="R5" library="rcl" library_urn="urn:adsk.eagle:library:334" deviceset="R-EU_" device="R1206" package3d_urn="urn:adsk.eagle:package:23540/2" value="1K"/>
+<part name="U$1" library="fab" library_urn="urn:adsk.eagle:library:9340542" deviceset="LED" device="FAB1206" package3d_urn="urn:adsk.eagle:package:9340753/2"/>
 </parts>
 <sheets>
@@
 <attribute name="VALUE" x="15.24" y="120.65" size="1.778" layer="96" rot="R90"/>
 </instance>
+<instance part="C2" gate="G$1" x="-7.62" y="106.68" smashed="yes">
+<attribute name="NAME" x="-6.477" y="107.1626" size="1.778" layer="95"/>
+<attribute name="VALUE" x="-6.477" y="102.0826" size="1.778" layer="96"/>
+</instance>
+<instance part="GND7" gate="1" x="111.76" y="73.66" smashed="yes">
+<attribute name="VALUE" x="109.22" y="71.12" size="1.778" layer="96"/>
+</instance>
+<instance part="R5" gate="G$1" x="111.76" y="93.98" smashed="yes" rot="R90">
+<attribute name="NAME" x="110.2614" y="90.17" size="1.778" layer="95" rot="R90"/>
+<attribute name="VALUE" x="115.062" y="90.17" size="1.778" layer="96" rot="R90"/>
+</instance>
+<instance part="U$1" gate="G$1" x="111.76" y="81.28" smashed="yes">
+<attribute name="NAME" x="115.316" y="79.248" size="1.778" layer="95" rot="R90"/>
+<attribute name="VALUE" x="117.475" y="79.248" size="1.778" layer="96" rot="R90"/>
+</instance>
 </instances>
 <busses>
@@
 <wire x1="5.08" y1="99.06" x2="0" y2="99.06" width="0.1524" layer="91"/>
 <junction x="0" y="99.06"/>
+<pinref part="C2" gate="G$1" pin="-"/>
+<wire x1="-7.62" y1="101.6" x2="-7.62" y2="99.06" width="0.1524" layer="91"/>
+<wire x1="-7.62" y1="99.06" x2="0" y2="99.06" width="0.1524" layer="91"/>
 </segment>
 <segment>
@@
 <pinref part="GND3" gate="1" pin="GND"/>
 <wire x1="30.48" y1="81.28" x2="30.48" y2="78.74" width="0.1524" layer="91"/>
+</segment>
+<segment>
+<pinref part="GND7" gate="1" pin="GND"/>
+<pinref part="U$1" gate="G$1" pin="C"/>
+<wire x1="111.76" y1="76.2" x2="111.76" y2="78.74" width="0.1524" layer="91"/>
 </segment>
 </net>
@@
 <wire x1="5.08" y1="114.3" x2="0" y2="114.3" width="0.1524" layer="91"/>
 <junction x="0" y="114.3"/>
+<pinref part="C2" gate="G$1" pin="+"/>
+<wire x1="-7.62" y1="109.22" x2="-7.62" y2="114.3" width="0.1524" layer="91"/>
+<wire x1="-7.62" y1="114.3" x2="0" y2="114.3" width="0.1524" layer="91"/>
 </segment>
 <segment>
@@
 </segment>
 </net>
+<net name="N$6" class="0">
+<segment>
+<pinref part="U$1" gate="G$1" pin="A"/>
+<pinref part="R5" gate="G$1" pin="1"/>
+<wire x1="111.76" y1="86.36" x2="111.76" y2="88.9" width="0.1524" layer="91"/>
+</segment>
+</net>
+<net name="N$7" class="0">
+<segment>
+<pinref part="IC1" gate="G$1" pin="(LUT0-IN1/TCA0WO1/SDA/MOSI/AIN1)PA1"/>
+<pinref part="R5" gate="G$1" pin="2"/>
+<wire x1="104.14" y1="101.6" x2="111.76" y2="101.6" width="0.1524" layer="91"/>
+<wire x1="111.76" y1="101.6" x2="111.76" y2="99.06" width="0.1524" layer="91"/>
+</segment>
+</net>
